File: FIC-100A.kicad_pcb (KiCad board)
At the start: 2 copper layers, 40 x 25 mm, 40 parts, among them J1 USB4105-GF-A, Q1 PT334-6C, U1 LM393, U2 USBLC6-2SC6, U3 FT231XS-U

Commit message: chore: snapshot project before Boardwright migration
Parts:
- moved TP2 0.50 mm to (131.0, 94.5)
Routing:
- net /CIRCUIT/TX: track 19.8 -> 25.5 mm
- net /CIRCUIT/RX: track 38.2 -> 41.4 mm
- net +3V3: track 46.4 -> 45.9 mm
- net GND: vias 52 -> 56
