File: FIC-100A.kicad_pcb (KiCad board)
At the start: 2 copper layers, 40 x 25 mm, 40 parts, among them J1 USB4105-GF-A, Q1 PT334-6C, U1 LM393, U2 USBLC6-2SC6, U3 FT231XS-U

Commit message: feat: migrate project to Boardwright
Parts:
- moved TP2 0.50 mm to (131.0, 94.5)
Routing:
- net /CIRCUIT/TX: track 19.8 -> 25.5 mm
- net /CIRCUIT/RX: track 38.2 -> 41.4 mm
- net +3V3: track 46.4 -> 45.9 mm
- net GND: vias 52 -> 56
Other:
- board text added: "0.02mm"
- board text added: "0.035mm (1.00oz)"
- board text added: "1.49mm"
- board text added: "B.Mask"
- board text added: "B.Paste"
- board text added: "B.Silkscreen"
- board text added: "Copper"
- board text added: "Core"
- board text added: "Dielectric"
- board text added: "Direct Printing"
- board text added: "F.Mask"
- board text added: "F.Paste"
- board text added: "F.Silkscreen"
- board text added: "FR4_7628"
- board text added: "GBR"
- board text added: "Gerber"
- board text added: "L1 (Sig, PWR)"
- board text added: "L2 (Sig, GND)"
- board text added: "Layer"
- board text added: "Legend"
- board text added: "Material"
- board text added: "Note: external layer thicknesses are specified after plating"
- board text added: "Paste Mask"
- board text added: "Plane"
- board text added: "Signal"
- board text added: "Solder Mask"
- board text added: "Solder Resist"
- board text added: "Thickness"
- board text added: "Total thickness: 1.6mm"
- board text added: "Type"
