File: FIC-100A.kicad_sch (KiCad schematic)
At the start: 0 parts

Commit message: feat: migrate project to Boardwright
Other:
- removed sheet REVISION HISTORY
- note added: "${PCBA_NAME} / ${PCB_NAME}"
- note added: "REV ${DRAWING_REVISION}"
- note removed: "${BOARD_NAME}"
- note removed: "DESIGN CONSIDERATIONS"
- note removed: "REV ${REVISION}"
